File: pcb/sparse-conv-host/mcu.kicad_sch (KiCad schematic)
At the start: 35 parts, among them J2 SWD, SW1 BOOT, SW2 RESET, U2 RP2350B, U3 W25Q32JVSS, Y1 12MHz

Commit message: Host board: bundle the two footprints KiCad 9 lacks
KiCad 9's ERC found no errors, but L_2016X120N (RP2350 core-regulator
inductor, from the demo board's private library) and VSSOP-10_3x3mm_P0.5mm
(INA228) were not in its standard libraries. Both now live in the project's
SparseConvHost.pretty. Netlist and footprint checks pass.

Co-Authored-By: Claude Opus 5.5 <noreply@anthropic.com>
Claude-Session: https://claude.ai/code/session_01WuUZbH4cddB8o6Ya7TKaqN
Parts:
- L1: footprint Inductor_SMD:L_2016X120N -> SparseConvHost:L_2016X120N
Changed lines of the file:
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@@
       )
     )
-    (property "Footprint" "Inductor_SMD:L_2016X120N"
+    (property "Footprint" "SparseConvHost:L_2016X120N"
       (at 134.62 96.52 0)
       (effects
