File: pcb/sparse-conv-host/power_monitor.kicad_sch (KiCad schematic)
At the start: 12 parts, among them J8 CORE, J9 RANGE, U4 INA228

Commit message: Host board: bundle the two footprints KiCad 9 lacks
KiCad 9's ERC found no errors, but L_2016X120N (RP2350 core-regulator
inductor, from the demo board's private library) and VSSOP-10_3x3mm_P0.5mm
(INA228) were not in its standard libraries. Both now live in the project's
SparseConvHost.pretty. Netlist and footprint checks pass.

Co-Authored-By: Claude Opus 5.5 <noreply@anthropic.com>
Claude-Session: https://claude.ai/code/session_01WuUZbH4cddB8o6Ya7TKaqN
Parts:
- U4: footprint Package_SO:VSSOP-10_3x3mm_P0.5mm -> SparseConvHost:VSSOP-10_3x3mm_P0.5mm
Changed lines of the file:
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@@
       )
     )
-    (property "Footprint" "Package_SO:VSSOP-10_3x3mm_P0.5mm"
+    (property "Footprint" "SparseConvHost:VSSOP-10_3x3mm_P0.5mm"
       (at 213.36 50.8 0)
       (effects
